Commit message: Lower casters by 10 mm
Wheel bottoms were previously 10 mm above base_link. With base_link
along the ground plane, wheels would hover 10 mm above the ground,
which caused the robot to fall at the start of physics simulations.

This change is consistent with physical wheel and chassis measurements.
Wheel axles are now at Z = 90 mm and wheel bottoms at Z = 0 relative to
base_link.

File: robot_model/xacros/mpo_700_body.urdf.xacro (robot description, xacro)
@@ -57,5 +57,5 @@
       link_origin_rpy="0 0 ${3.14 * angle_comp}"
       >
-      <origin rpy="0 0 0" xyz="0.24 0.18 0.22"/>
+      <origin rpy="0 0 0" xyz="0.24 0.18 0.21"/>
     </xacro:mpo_700_caster_wheel>
     <xacro:mpo_700_caster_wheel
@@ -65,5 +65,5 @@
       link_origin_rpy="0 0 3.14"
       >
-      <origin rpy="0 0 0" xyz="0.24 -0.18 0.22"/>
+      <origin rpy="0 0 0" xyz="0.24 -0.18 0.21"/>
     </xacro:mpo_700_caster_wheel>
     <xacro:mpo_700_caster_wheel
@@ -73,5 +73,5 @@
       link_origin_rpy="0 0 ${3.14 * angle_comp}"
       >
-      <origin rpy="0 0 0" xyz="-0.24 0.18 0.22"/>
+      <origin rpy="0 0 0" xyz="-0.24 0.18 0.21"/>
     </xacro:mpo_700_caster_wheel>
     <xacro:mpo_700_caster_wheel
@@ -81,5 +81,5 @@
       link_origin_rpy="0 0 3.14"
       >
-      <origin rpy="0 0 0" xyz="-0.24 -0.18 0.22"/>
+      <origin rpy="0 0 0" xyz="-0.24 -0.18 0.21"/>
     </xacro:mpo_700_caster_wheel>
     <!-- Wheels -->

Commit message: Move casters outward by 10 mm
Caster steering axes were 360 mm apart laterally in the model, compared
to 380 mm measured on the physical robot and specified in the kinematics
configuration. This change also corrects the spacing between left/right
wheel centers in the model to the measured 470 mm on the physical robot
in the outward home arrangement.

File: robot_model/xacros/mpo_700_body.urdf.xacro (robot description, xacro)
@@ -57,5 +57,5 @@
       link_origin_rpy="0 0 ${3.14 * angle_comp}"
       >
-      <origin rpy="0 0 0" xyz="0.24 0.18 0.21"/>
+      <origin rpy="0 0 0" xyz="0.24 0.19 0.21"/>
     </xacro:mpo_700_caster_wheel>
     <xacro:mpo_700_caster_wheel
@@ -65,5 +65,5 @@
       link_origin_rpy="0 0 3.14"
       >
-      <origin rpy="0 0 0" xyz="0.24 -0.18 0.21"/>
+      <origin rpy="0 0 0" xyz="0.24 -0.19 0.21"/>
     </xacro:mpo_700_caster_wheel>
     <xacro:mpo_700_caster_wheel
@@ -73,5 +73,5 @@
       link_origin_rpy="0 0 ${3.14 * angle_comp}"
       >
-      <origin rpy="0 0 0" xyz="-0.24 0.18 0.21"/>
+      <origin rpy="0 0 0" xyz="-0.24 0.19 0.21"/>
     </xacro:mpo_700_caster_wheel>
     <xacro:mpo_700_caster_wheel
@@ -81,5 +81,5 @@
       link_origin_rpy="0 0 3.14"
       >
-      <origin rpy="0 0 0" xyz="-0.24 -0.18 0.21"/>
+      <origin rpy="0 0 0" xyz="-0.24 -0.19 0.21"/>
     </xacro:mpo_700_caster_wheel>
     <!-- Wheels -->
